File: kicad_lorenz/kicad_lorenz.kicad_pcb (KiCad board)
At the start: 2 copper layers, 105 x 90 mm, 39 parts, among them J1 X,-Y,Z, J2 Power_In, M2 MountingHole_2.2mm_M2, SW1 SW_DIP_x09, U1 TL074, U2 AD633JN, U3 AD633JN, U4 TPS65131

Commit message: with traces
Parts:
- moved C15 10.7 mm to (112.9, 106.3), turned to -90 degrees
- moved C6 9.84 mm to (119.3, 114.6), turned to 0 degrees
- moved C5 2.02 mm to (114.0, 75.3), turned to -90 degrees
- moved R4 0.42 mm to (85.0, 88.5)
- moved R1 0.28 mm to (85.0, 84.3)
Routing:
- net +15V: track 0.00 -> 147.4 mm, vias 0 -> 1
- net -15V: track 0.00 -> 141.9 mm, vias 0 -> 2
- net Net-(J1-Pin_1): track 33.4 -> 150.2 mm
- net Net-(J1-Pin_3): track 22.4 -> 133.2 mm, vias 0 -> 2
- net Net-(J1-Pin_2): track 20.0 -> 130.0 mm, vias 0 -> 1
- net Net-(U1C--): track 28.4 -> 86.2 mm
- net Net-(U1B--): track 13.0 -> 61.9 mm
- net Net-(U1A--): track 12.8 -> 59.6 mm
- net Net-(C11-Pad1): track 0.00 -> 45.6 mm, vias 0 -> 1
- net Net-(C1-Pad1): track 0.00 -> 44.0 mm
- net Net-(C8-Pad1): track 0.00 -> 37.3 mm
- net Net-(C12-Pad1): track 0.00 -> 36.0 mm, vias 0 -> 1
- net Net-(U3-W): track 0.00 -> 35.9 mm
- net Net-(C2-Pad1): track 0.00 -> 34.1 mm
- net Net-(C9-Pad1): track 0.00 -> 31.4 mm
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
Commit message: DIP Switch Layout instructions
Parts:
- DiffEq_F_Out: renamed from J1; value X,-Y,Z -> X -Y Z
- GND  3-5.5V: renamed from J2
Other:
- board text added: "DIP Switch Layout Z: Fast (2n) Med Slow Y: Fast Med (0.1u) Slow X: Fast Med Slow (0.47u)"
Changed lines of the file:
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@@
 		(descr "Soldered wire connection, for 3 times 0.5 mm² wires, reinforced insulation, conductor diameter 0.9mm, outer diameter 2.3mm, size source Multi-Contact FLEXI-xV 0.50 (https://www.staubli.com/content/dam/ecs/catalogs-brochures/TM/CAB-Main-11014119-en.pdf#page=11), bend radius 3 times outer diameter")
 		(tags "connector wire 0.5sqmm")
-		(property "Reference" "J1"
+		(property "Reference" "DiffEq_F_Out"
 			(at 4.8 -2.35 90)
 			(layer "F.SilkS")
@@
 			)
 		)
-		(property "Value" "X,-Y,Z"
+		(property "Value" "X    -Y    Z"
 			(at 4.8 2.35 90)
 			(layer "F.SilkS")
@@
 		(descr "Soldered wire connection, for 2 times 0.5 mm² wires, reinforced insulation, conductor diameter 0.9mm, outer diameter 2.3mm, size source Multi-Contact FLEXI-xV 0.50 (https://www.staubli.com/content/dam/ecs/catalogs-brochures/TM/CAB-Main-11014119-en.pdf#page=11), bend radius 3 times outer diameter")
 		(tags "connector wire 0.5sqmm")
-		(property "Reference" "J2"
+		(property "Reference" "GND  3-5.5V"
 			(at 2.4 -2.35 0)
 			(layer "F.SilkS")
@@
 		(layer "F.SilkS")
 		(effects
+			(font
+				(size 1 1)
+				(thickness 0.15)
+			)
+			(justify left bottom)
+		)
+	)
+	(gr_text "DIP Switch Layout\nZ:  Fast (2n)\n    Med\n    Slow\nY:  Fast\n    Med  (0.1u)\n    Slow\nX:  Fast\n    Med\n    Slow (0.47u)"
+		(at 144.5 96.9 0)
+		(layer "F.SilkS")
+		(effects
